File: Logiplant/Logiplant/Logiplant.kicad_pcb (KiCad board)
At the start: 2 copper layers, 104.2 x 116 mm, 16 parts, among them J4 POWER, J6 Conn_RELE, J7 Conn_IMPRESOR, U2 ESP32-DEVKITC-32D

Commit message: Cambio de oled
Parts:
- moved OLED1 9.11 mm to (-97.0, 80.5)

Commit message: Nueva regulación
Parts:
- removed R2: 1K, Resistor_THT:R_Axial_DIN0207_L6.3mm_D2.5mm_P5.08mm_Vertical
- removed R3: 2.2K, Resistor_THT:R_Axial_DIN0207_L6.3mm_D2.5mm_P5.08mm_Vertical
- added U1: LD1117S33TR_SOT223, Package_TO_SOT_THT:TO-220-3_Vertical, F.Cu at (-123.4, 162.1)
- added U3: LM7805_TO220, Package_TO_SOT_THT:TO-220-3_Vertical, F.Cu at (-123.0, 180.1)
- R4: footprint Resistor_THT:R_Axial_DIN0207_L6.3mm_D2.5mm_P10.16mm_Horizontal -> Resistor_THT:R_Axial_DIN0207_L6.3mm_D2.5mm_P5.08mm_Vertical
Connections:
- J4 pad 2: +5V -> Net-(J4-Pad2)
Routing:
- net +5V: track 196.4 -> 227.7 mm
- net Net-(J4-Pad2): track 0.00 -> 16.3 mm
- net +3V3: track 184.9 -> 187.4 mm
- net IO21: track 42.7 -> 44.6 mm
Other:
- board size 104.2 x 116 mm -> 100.4 x 116 mm

Commit message: Nuevo prog
Parts:
- removed J6: Conn_RELE, MODULOS:ReleYYG
- removed J7: Conn_IMPRESOR, TerminalBlock_Phoenix:TerminalBlock_Phoenix_MKDS-1,5-3-5.08_1x03_P5.08mm_Horizontal
- removed R4: 1k, Resistor_THT:R_Axial_DIN0207_L6.3mm_D2.5mm_P5.08mm_Vertical
- added U4: TarjetaRele, MODULOS:ReleYYG, F.Cu at (-2.06, 149.1)
- Recibo1: value Conn_01x02 -> Conn_01x03; footprint Connector_PinHeader_2.54mm:PinHeader_1x02_P2.54mm_Vertical -> TerminalBlock_Phoenix:TerminalBlock_Phoenix_MKDS-1,5-3-5.08_1x03_P5.08mm_Horizontal
- moved OLED1 70.5 mm to (-50.6, 133.6), turned to 90 degrees
- moved HALL1 64.2 mm to (-125.9, 107.9)
- moved Recibo1 52.5 mm to (-114.5, 67.9), turned to 180 degrees
- moved D1 47.5 mm to (-70.4, 141.8)
- moved U2 18.3 mm to (-98.6, 124.3), turned to 90 degrees
Connections:
- J4 pad 2: Net-(J4-Pad2) -> +12V
- Recibo1 pad 1: IO25 -> GND
- Recibo1 pad 2: +3V3 -> +12V
- U3 pad 1: Net-(J4-Pad2) -> +12V
Routing:
- net +5V: track 227.7 -> 0.00 mm
- net +3V3: track 187.4 -> 0.00 mm
- net IO25: track 81.1 -> 0.00 mm
- net IO27: track 59.5 -> 0.00 mm
- net IO26: track 58.6 -> 0.00 mm
- net IO21: track 44.6 -> 0.00 mm
- net MOSI-DATA: track 44.0 -> 0.00 mm
- net IO33: track 43.9 -> 0.00 mm
- net CD-DC: track 36.8 -> 0.00 mm
- net RST: track 36.1 -> 0.00 mm
- net SCK: track 33.2 -> 0.00 mm
- net CS: track 27.1 -> 0.00 mm
- net IO18: track 23.6 -> 0.00 mm
- net IO19: track 20.7 -> 0.00 mm
- net Net-(J4-Pad2): track 16.3 -> 0.00 mm

Commit message: Nuevo circuito
Nuevo circuito
Parts:
- added R2: 0, Resistor_THT:R_Axial_DIN0207_L6.3mm_D2.5mm_P10.16mm_Horizontal, F.Cu at (-112.0, 111.0)
- added R3: 0, Resistor_THT:R_Axial_DIN0207_L6.3mm_D2.5mm_P10.16mm_Horizontal, F.Cu at (-79.8, 179.8)
- moved U4 113.6 mm to (-102.1, 95.2), turned to 270 degrees
- moved R1 76.7 mm to (-49.4, 127.2), turned to 180 degrees
- moved Bolsa1 68.6 mm to (-54.4, 132.6), turned to 90 degrees
- moved R5 64.0 mm to (-65.1, 124.0), turned to 270 degrees
- moved Recibo1 62.5 mm to (-126.1, 129.4), turned to 270 degrees
- moved Seguro1 58.7 mm to (-65.1, 132.8), turned to 90 degrees
- moved SERVO1 54.7 mm to (-72.0, 133.1), turned to 270 degrees
- moved OLED1 28.2 mm to (-48.9, 161.8)
- moved U2 27.5 mm to (-98.8, 151.8)
- moved D1 26.5 mm to (-68.7, 168.2)
- moved U1 21.2 mm to (-114.0, 181.2), turned to 180 degrees
- moved HALL1 13.1 mm to (-118.8, 118.9), turned to 180 degrees
- moved J4 6.63 mm to (-106.6, 185.7)
- moved U3 5.83 mm to (-126.1, 185.0)
Connections:
- U4 pad 4: +12V -> Net-(U4-Pad4)
Routing:
- net +3V3: track 0.00 -> 273.8 mm
- net +12V: track 0.00 -> 146.9 mm
- net IO26: track 0.00 -> 83.0 mm
- net +5V: track 0.00 -> 67.6 mm
- net IO18: track 0.00 -> 50.1 mm
- net IO33: track 0.00 -> 46.6 mm
- net CS: track 0.00 -> 40.4 mm
- net IO19: track 0.00 -> 35.9 mm
- net IO25: track 0.00 -> 21.3 mm
- net GND: track 0.00 -> 20.9 mm
- net CD-DC: track 0.00 -> 20.4 mm
- net IO21: track 0.00 -> 13.9 mm
- net MOSI-DATA: track 0.00 -> 12.0 mm
- net RST: track 0.00 -> 11.4 mm
- net SCK: track 0.00 -> 11.0 mm

Commit message: Cambios PCB
Parts:
- U4: footprint MODULOS:ReleYYG -> TerminalBlock_Phoenix:TerminalBlock_Phoenix_MKDS-1,5-3-5.08_1x03_P5.08mm_Horizontal
- moved J4 37.9 mm to (-126.5, 153.4), turned to 270 degrees
- moved U3 18.6 mm to (-122.0, 166.9), turned to 270 degrees
- moved U1 14.3 mm to (-127.0, 187.1), turned to 90 degrees
Connections:
- U2 pad 19: Net-(U2-Pad19) -> +5V
Routing:
- net +12V: track 146.9 -> 101.9 mm
- net +5V: track 67.6 -> 76.0 mm
- net +3V3: track 273.8 -> 277.9 mm
- net (no net): vias 0 -> 2
