File: Logiplant/Logiplant/Logiplant.sch (KiCad schematic (older format))
At the start: 18 parts, among them J4 POWER, J6 Conn_RELE, J7 Conn_IMPRESOR, U2 ESP32-DEVKITC-32D

Commit message: Nuevo prog
Parts:
- removed J6: Conn_RELE, MODULOS:ReleYYG, symbol Connector_Generic:Conn_01x03
- removed J7: Conn_IMPRESOR, TerminalBlock_Phoenix:TerminalBlock_Phoenix_MKDS-1,5-3-5.08_1x03_P5.08mm_Horizontal, symbol Connector_Generic:Conn_01x03
- removed R2: 1K, Resistor_THT:R_Axial_DIN0207_L6.3mm_D2.5mm_P5.08mm_Vertical, symbol Device:R
- removed R3: 2.2K, Resistor_THT:R_Axial_DIN0207_L6.3mm_D2.5mm_P5.08mm_Vertical, symbol Device:R
- removed R4: 1k, Resistor_THT:R_Axial_DIN0207_L6.3mm_D2.5mm_P5.08mm_Vertical, symbol Device:R
- removed Recibo1: Conn_01x02, Connector_PinHeader_2.54mm:PinHeader_1x02_P2.54mm_Vertical, symbol Connector_Generic:Conn_01x02
- added Recibo1: Conn_01x03, TerminalBlock_Phoenix:TerminalBlock_Phoenix_MKDS-1,5-3-5.08_1x03_P5.08mm_Horizontal, symbol Connector_Generic:Conn_01x03
- added U4: TarjetaRele, MODULOS:ReleYYG, symbol TarjetaRele:TarjetaRele
- U1: renamed from U?; footprint Package_TO_SOT_SMD:SOT-223-3_TabPin2 -> Package_TO_SOT_THT:TO-220-3_Vertical
- gave numbers to parts that had none: 1
Connections:
- net labels added: +12V
- wire segments 21 -> 10
- no-connect marks 0 -> 2
Other:
- note added: "FUENTE"
- moved on the sheet: Bolsa1, D1, HALL1, J4, OLED1, R1, R5, SERVO1, Seguro1, U1, U3

Commit message: Nuevo circuito
Nuevo circuito
Parts:
- added R2, R3: 0, Resistor_THT:R_Axial_DIN0207_L6.3mm_D2.5mm_P5.08mm_Vertical, symbol Device:R
Connections:
- net +12V: no longer U4.4 (COM)
- net GND: now also R2.1, R2.2, R3.1, R3.2
- no-connect marks 2 -> 3
Changed lines of the file:
@@
 NoConn ~ 2000 2400
-$Comp
-L power:+12V #PWR0129
-U 1 1 653AE45F
-P 2000 2300
-F 0 "#PWR0129" H 2000 2150 50  0001 C CNN
-F 1 "+12V" V 2015 2428 50  0000 L CNN
-F 2 "" H 2000 2300 50  0001 C CNN
-F 3 "" H 2000 2300 50  0001 C CNN
-	1    2000 2300
-	0    1    1    0
-$EndComp
 $Comp
 L Connector_Generic:Conn_01x03 Recibo1
@@
 	-1   0    0    1
 $EndComp
+NoConn ~ 2000 2300
+$Comp
+L Device:R R3
+U 1 1 65436935
+P 6350 3150
+F 0 "R3" V 6143 3150 50  0000 C CNN
+F 1 "0" V 6234 3150 50  0000 C CNN
+F 2 "Resistor_THT:R_Axial_DIN0207_L6.3mm_D2.5mm_P5.08mm_Vertical" V 6280 3150 50  0001 C CNN
+F 3 "~" H 6350 3150 50  0001 C CNN
+	1    6350 3150
+	0    1    -1   0
+$EndComp
+$Comp
+L Device:R R2
+U 1 1 654370B9
+P 6350 2950
+F 0 "R2" V 6143 2950 50  0000 C CNN
+F 1 "0" V 6234 2950 50  0000 C CNN
+F 2 "Resistor_THT:R_Axial_DIN0207_L6.3mm_D2.5mm_P5.08mm_Vertical" V 6280 2950 50  0001 C CNN
+F 3 "~" H 6350 2950 50  0001 C CNN
+	1    6350 2950
+	0    -1   1    0
+$EndComp
+$Comp
+L power:GND #PWR0120
+U 1 1 6543798B
+P 6200 2950
+F 0 "#PWR0120" H 6200 2700 50  0001 C CNN
+F 1 "GND" H 6205 2777 50  0000 C CNN
+F 2 "" H 6200 2950 50  0001 C CNN
+F 3 "" H 6200 2950 50  0001 C CNN
+	1    6200 2950
+	0    1    1    0
+$EndComp
+$Comp
+L power:GND #PWR0127
+U 1 1 65438E79
+P 6500 3150
+F 0 "#PWR0127" H 6500 2900 50  0001 C CNN
+F 1 "GND" H 6505 2977 50  0000 C CNN
+F 2 "" H 6500 3150 50  0001 C CNN
+F 3 "" H 6500 3150 50  0001 C CNN
+	1    6500 3150
+	0    -1   1    0
+$EndComp
+Wire Wire Line
+	6500 2950 6500 3150
+Connection ~ 6500 3150
+Wire Wire Line
+	6200 3150 6200 2950
+Connection ~ 6200 2950
 $EndSCHEMATC

Commit message: Cambios PCB
Parts:
- R2, R3: footprint Resistor_THT:R_Axial_DIN0207_L6.3mm_D2.5mm_P5.08mm_Vertical -> Resistor_THT:R_Axial_DIN0207_L6.3mm_D2.5mm_P10.16mm_Horizontal
- U4: footprint MODULOS:ReleYYG -> TerminalBlock_Phoenix:TerminalBlock_Phoenix_MKDS-1,5-3-5.08_1x03_P5.08mm_Horizontal
Connections:
- net +5V: now also U2.19 (EXT_5V)
Changed lines of the file:
@@
 F 0 "U4" H 1475 2725 50  0000 C CNN
 F 1 "TarjetaRele" H 1475 2634 50  0000 C CNN
-F 2 "MODULOS:ReleYYG" H 1450 2600 50  0001 C CNN
+F 2 "TerminalBlock_Phoenix:TerminalBlock_Phoenix_MKDS-1,5-3-5.08_1x03_P5.08mm_Horizontal" H 1450 2600 50  0001 C CNN
 F 3 "" H 1480 2680 50  0001 C CNN
 	1    1450 2400
@@
 F 0 "R3" V 6143 3150 50  0000 C CNN
 F 1 "0" V 6234 3150 50  0000 C CNN
-F 2 "Resistor_THT:R_Axial_DIN0207_L6.3mm_D2.5mm_P5.08mm_Vertical" V 6280 3150 50  0001 C CNN
+F 2 "Resistor_THT:R_Axial_DIN0207_L6.3mm_D2.5mm_P10.16mm_Horizontal" V 6280 3150 50  0001 C CNN
 F 3 "~" H 6350 3150 50  0001 C CNN
 	1    6350 3150
@@
 F 0 "R2" V 6143 2950 50  0000 C CNN
 F 1 "0" V 6234 2950 50  0000 C CNN
-F 2 "Resistor_THT:R_Axial_DIN0207_L6.3mm_D2.5mm_P5.08mm_Vertical" V 6280 2950 50  0001 C CNN
+F 2 "Resistor_THT:R_Axial_DIN0207_L6.3mm_D2.5mm_P10.16mm_Horizontal" V 6280 2950 50  0001 C CNN
 F 3 "~" H 6350 2950 50  0001 C CNN
 	1    6350 2950
@@
 	6200 3150 6200 2950
 Connection ~ 6200 2950
+$Comp
+L power:+5V #PWR0129
+U 1 1 655E37FF
+P 5550 2550
+F 0 "#PWR0129" H 5550 2400 50  0001 C CNN
+F 1 "+5V" V 5565 2678 50  0000 L CNN
+F 2 "" H 5550 2550 50  0001 C CNN
+F 3 "" H 5550 2550 50  0001 C CNN
+	1    5550 2550
+	0    -1   -1   0
+$EndComp
 $EndSCHEMATC
