File: Logiplant/LogiGSM/LogiGSM.sch (EAGLE design)
At the start: 17 parts, among them IC1 7805TV, IC2 LM1117T-3.3-V

Commit message: Problemas con interrupcion
Problemas con interrupcion
Parts:
- renumbered JP1 to GSM
Other:
- moved on the sheet: CABLE
Changed lines of the file:
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@@
 <part name="P+4" library="supply1" library_urn="urn:adsk.eagle:library:371" deviceset="+12V" device=""/>
 <part name="P+5" library="supply1" library_urn="urn:adsk.eagle:library:371" deviceset="+5V" device=""/>
-<part name="P+6" library="supply1" library_urn="urn:adsk.eagle:library:371" deviceset="+5V" device=""/>
+<part name="P+6" library="supply1" library_urn="urn:adsk.eagle:library:371" deviceset="+5V" device="" value="+4V7"/>
 <part name="+3V7" library="supply1" library_urn="urn:adsk.eagle:library:371" deviceset="+3V3" device=""/>
 <part name="GND1" library="supply1" library_urn="urn:adsk.eagle:library:371" deviceset="GND" device=""/>
@@
 <part name="GND13" library="supply1" library_urn="urn:adsk.eagle:library:371" deviceset="GND" device=""/>
 <part name="CABLE" library="resistor-power" deviceset="R" device="RS1/2" package3d_urn="urn:adsk.eagle:package:25166/1" value="0k"/>
-<part name="JP1" library="pinhead" library_urn="urn:adsk.eagle:library:325" deviceset="PINHD-1X6" device="" package3d_urn="urn:adsk.eagle:package:22472/2"/>
+<part name="GSM" library="pinhead" library_urn="urn:adsk.eagle:library:325" deviceset="PINHD-1X6" device="" package3d_urn="urn:adsk.eagle:package:22472/2"/>
 <part name="P+7" library="supply1" library_urn="urn:adsk.eagle:library:371" deviceset="+5V" device=""/>
 <part name="GND14" library="supply1" library_urn="urn:adsk.eagle:library:371" deviceset="GND" device=""/>
@@
 <attribute name="VALUE" x="577.85" y="-491.363" size="1.778" layer="96" rot="MR0"/>
 </instance>
-<instance part="GND12" gate="1" x="614.68" y="-556.26" smashed="yes" rot="R270">
-<attribute name="VALUE" x="609.6" y="-556.26" size="1.778" layer="96"/>
-</instance>
-<instance part="GND13" gate="1" x="629.92" y="-556.26" smashed="yes" rot="R90">
-<attribute name="VALUE" x="635" y="-556.26" size="1.778" layer="96" rot="R180"/>
-</instance>
-<instance part="CABLE" gate="G$1" x="622.3" y="-556.26" smashed="yes">
-<attribute name="NAME" x="618.49" y="-554.8884" size="1.778" layer="95"/>
-<attribute name="VALUE" x="618.49" y="-559.181" size="1.778" layer="96"/>
-</instance>
-<instance part="JP1" gate="A" x="703.58" y="-482.6" smashed="yes">
+<instance part="GND12" gate="1" x="612.14" y="-487.68" smashed="yes" rot="R270">
+<attribute name="VALUE" x="607.06" y="-487.68" size="1.778" layer="96"/>
+</instance>
+<instance part="GND13" gate="1" x="627.38" y="-487.68" smashed="yes" rot="R90">
+<attribute name="VALUE" x="632.46" y="-487.68" size="1.778" layer="96" rot="R180"/>
+</instance>
+<instance part="CABLE" gate="G$1" x="619.76" y="-487.68" smashed="yes">
+<attribute name="NAME" x="615.95" y="-486.3084" size="1.778" layer="95"/>
+<attribute name="VALUE" x="615.95" y="-490.601" size="1.778" layer="96"/>
+</instance>
+<instance part="GSM" gate="A" x="703.58" y="-482.6" smashed="yes">
 <attribute name="NAME" x="697.23" y="-471.805" size="1.778" layer="95"/>
 <attribute name="VALUE" x="697.23" y="-492.76" size="1.778" layer="96"/>
@@
 <segment>
 <pinref part="GND14" gate="1" pin="GND"/>
-<pinref part="JP1" gate="A" pin="6"/>
+<pinref part="GSM" gate="A" pin="6"/>
 <wire x1="690.88" y1="-487.68" x2="701.04" y2="-487.68" width="0.1524" layer="91"/>
 </segment>
@@
 <net name="N$1" class="0">
 <segment>
-<pinref part="JP1" gate="A" pin="2"/>
+<pinref part="GSM" gate="A" pin="2"/>
 <wire x1="693.42" y1="-477.52" x2="701.04" y2="-477.52" width="0.1524" layer="91"/>
 <pinref part="D2" gate="G$1" pin="A"/>
@@
 <net name="RXD" class="0">
 <segment>
-<pinref part="JP1" gate="A" pin="4"/>
+<pinref part="GSM" gate="A" pin="4"/>
 <wire x1="701.04" y1="-482.6" x2="695.96" y2="-482.6" width="0.1524" layer="91"/>
 <label x="695.96" y="-482.6" size="1.27" layer="95" rot="R180" xref="yes"/>
@@
 <net name="TXD" class="0">
 <segment>
-<pinref part="JP1" gate="A" pin="5"/>
+<pinref part="GSM" gate="A" pin="5"/>
 <wire x1="701.04" y1="-485.14" x2="695.96" y2="-485.14" width="0.1524" layer="91"/>
 <label x="695.96" y="-485.14" size="1.27" layer="95" rot="R180" xref="yes"/>
@@
 <net name="NET" class="0">
 <segment>
-<pinref part="JP1" gate="A" pin="1"/>
+<pinref part="GSM" gate="A" pin="1"/>
 <wire x1="701.04" y1="-474.98" x2="695.96" y2="-474.98" width="0.1524" layer="91"/>
 <label x="695.96" y="-474.98" size="1.27" layer="95" rot="R180" xref="yes"/>
@@
 <net name="RST2" class="0">
 <segment>
-<pinref part="JP1" gate="A" pin="3"/>
+<pinref part="GSM" gate="A" pin="3"/>
 <wire x1="701.04" y1="-480.06" x2="695.96" y2="-480.06" width="0.1524" layer="91"/>
 <label x="695.96" y="-480.06" size="1.27" layer="95" rot="R180" xref="yes"/>
@@
 </sheet>
 </sheets>
+<errors>
+</errors>
 </schematic>
 </drawing>
