File: Logiplant/LogiGSMPCB/LogiGSM.brd (EAGLE design)
At the start: 123.2 x 82.7 mm, 17 parts, among them IC1 7805TV, IC2 LM1117T-3.3-V

Commit message: 28/11/2024
28/11/2024 Cambios en circuito
Parts:
- moved SERVO 80.3 mm to (85.1, 62.2)
- moved OLED 61.1 mm to (21.6, 22.9)
- moved CABLE 57.3 mm to (2.92, 65.5), turned to 269.5 degrees
- moved GSM 33.2 mm to (83.8, 20.3)
- moved D1 13.5 mm to (82.5, 7.62), turned to 180 degrees
- moved D2 13.0 mm to (99.1, 10.2)
- moved SHALL 12.0 mm to (14.0, 47.0), turned to 270 degrees
- moved R1 10.2 mm to (71.1, 43.2)
- moved RELEE 7.73 mm to (27.9, 62.2)
- moved IC1 7.62 mm to (3.81, 21.6)
- moved BOLSA 5.08 mm to (91.4, 50.8)
- moved SEGURO 5.08 mm to (77.5, 50.8)
- moved R2 4.58 mm to (85.1, 43.2)
Connections:
- removed net IO27: U$1.GPIO27
- net +3V3: now also SERVO.2, SHALL.2; no longer SERVO.1, SHALL.1
- net CD-DC: now also U$1.GPIO13; no longer U$1.GPIO16
- net CS: now also U$1.GPIO12; no longer U$1.GPIO0
- net IO21: now also SERVO.1; no longer SERVO.2
- net IO26: now also SHALL.1, U$1.GPIO32; no longer SHALL.2, U$1.GPIO26
- net MOSI-DATA: now also U$1.GPIO26; no longer U$1.GPIO17
- net RST: now also U$1.GPIO27; no longer U$1.GPIO2
- net RXD: now also U$1.GPIO17; no longer U$1.TX
- net SCK: now also U$1.GPIO14; no longer U$1.GPIO4
- net TXD: now also U$1.GPIO16; no longer U$1.RX
Routing:
- net +3V3: track 190.3 -> 344.7 mm
- net IO21: track 113.6 -> 41.3 mm
- net IO25: track 105.4 -> 46.7 mm
- net RXD: track 71.5 -> 23.2 mm
- net TXD: track 59.1 -> 23.2 mm
- net CD-DC: track 42.3 -> 15.8 mm
- net RST: track 35.9 -> 15.8 mm
- net IO26: track 69.5 -> 51.4 mm
- net IO33: track 55.3 -> 46.1 mm
- net +5V: track 215.9 -> 207.1 mm
- net N$1: track 30.8 -> 22.3 mm
- net MOSI-DATA: track 35.0 -> 27.7 mm
- net CS: track 21.4 -> 15.8 mm
- net IO19: track 26.2 -> 31.8 mm
- net SCK: track 20.3 -> 15.8 mm
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