File: Logiplant/LogiGSMPCB/LogiGSM.sch (EAGLE design)
At the start: 17 parts, among them IC1 7805TV, IC2 LM1117T-3.3-V

Commit message: 28/11/2024
28/11/2024 Cambios en circuito
Connections:
- removed net IO27: U$1.GPIO27(ADC2_7)
- net +3V3: now also SERVO.2, SHALL.2; no longer SERVO.1, SHALL.1
- net CD-DC: now also U$1.GPIO13(ADC2_4/MTCK/HSPI_MOSI); no longer U$1.GPIO16
- net CS: now also U$1.GPIO12(ADC2_5/MTDI/HSPI_MISO); no longer U$1.GPIO0(ADC2_1)
- net IO21: now also SERVO.1; no longer SERVO.2
- net IO26: now also SHALL.1, U$1.GPIO32(ADC1_4); no longer SHALL.2, U$1.GPIO26(ADC2_9)
- net MOSI-DATA: now also U$1.GPIO26(ADC2_9); no longer U$1.GPIO17
- net RST: now also U$1.GPIO27(ADC2_7); no longer U$1.GPIO2(ADC2_2)
- net RXD: now also U$1.GPIO17; no longer U$1.GPIO01(TX)
- net SCK: now also U$1.GPIO14(ADC2_6/MTMSHSPI_SCK); no longer U$1.GPIO4(ADC2_0)
- net TXD: now also U$1.GPIO16; no longer U$1.GPIO03(RX)
Changed lines of the file:
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@@
 <part name="P+4" library="supply1" library_urn="urn:adsk.eagle:library:371" deviceset="+12V" device=""/>
 <part name="P+5" library="supply1" library_urn="urn:adsk.eagle:library:371" deviceset="+5V" device=""/>
-<part name="P+6" library="supply1" library_urn="urn:adsk.eagle:library:371" deviceset="+5V" device=""/>
+<part name="P+6" library="supply1" library_urn="urn:adsk.eagle:library:371" deviceset="+5V" device="" value="+4V7"/>
 <part name="+3V7" library="supply1" library_urn="urn:adsk.eagle:library:371" deviceset="+3V3" device=""/>
 <part name="GND1" library="supply1" library_urn="urn:adsk.eagle:library:371" deviceset="GND" device=""/>
@@
 <attribute name="VALUE" x="584.2" y="-495.3" size="1.778" layer="96"/>
 </instance>
-<instance part="+3V3" gate="G$1" x="601.98" y="-447.04" smashed="yes" rot="R90">
-<attribute name="VALUE" x="601.98" y="-444.5" size="1.778" layer="96" rot="R180"/>
-</instance>
-<instance part="+3V4" gate="G$1" x="632.46" y="-447.04" smashed="yes" rot="R90">
-<attribute name="VALUE" x="635" y="-444.5" size="1.778" layer="96" rot="R180"/>
+<instance part="+3V3" gate="G$1" x="604.52" y="-449.58" smashed="yes" rot="R90">
+<attribute name="VALUE" x="604.52" y="-449.58" size="1.778" layer="96" rot="R180"/>
+</instance>
+<instance part="+3V4" gate="G$1" x="635" y="-449.58" smashed="yes" rot="R90">
+<attribute name="VALUE" x="635" y="-449.58" size="1.778" layer="96" rot="R180"/>
 </instance>
 <instance part="+3V5" gate="G$1" x="614.68" y="-474.98" smashed="yes" rot="R90">
@@
 </segment>
 <segment>
-<pinref part="SHALL" gate="A" pin="1"/>
-<pinref part="+3V3" gate="G$1" pin="+3V3"/>
-<wire x1="609.6" y1="-447.04" x2="604.52" y2="-447.04" width="0.1524" layer="91"/>
-</segment>
-<segment>
-<pinref part="SERVO" gate="A" pin="1"/>
-<pinref part="+3V4" gate="G$1" pin="+3V3"/>
-<wire x1="640.08" y1="-447.04" x2="635" y2="-447.04" width="0.1524" layer="91"/>
-</segment>
-<segment>
 <pinref part="OLED" gate="A" pin="1"/>
 <wire x1="680.72" y1="-434.34" x2="662.94" y2="-434.34" width="0.1524" layer="91"/>
@@
 <pinref part="BOLSA" gate="G$1" pin="2"/>
 <wire x1="617.22" y1="-474.98" x2="622.3" y2="-474.98" width="0.1524" layer="91"/>
+</segment>
+<segment>
+<pinref part="+3V3" gate="G$1" pin="+3V3"/>
+<pinref part="SHALL" gate="A" pin="2"/>
+<wire x1="607.06" y1="-449.58" x2="609.6" y2="-449.58" width="0.1524" layer="91"/>
+</segment>
+<segment>
+<pinref part="+3V4" gate="G$1" pin="+3V3"/>
+<pinref part="SERVO" gate="A" pin="2"/>
+<wire x1="637.54" y1="-449.58" x2="640.08" y2="-449.58" width="0.1524" layer="91"/>
 </segment>
 </net>
@@
 </segment>
 <segment>
-<pinref part="U$1" gate="G$1" pin="GPIO2(ADC2_2)"/>
-<wire x1="655.32" y1="-530.86" x2="665.48" y2="-530.86" width="0.1524" layer="91"/>
-<label x="665.48" y="-530.86" size="1.27" layer="95" xref="yes"/>
+<pinref part="U$1" gate="G$1" pin="GPIO27(ADC2_7)"/>
+<wire x1="589.28" y1="-520.7" x2="584.2" y2="-520.7" width="0.1524" layer="91"/>
+<label x="584.2" y="-520.7" size="1.016" layer="95" rot="R180" xref="yes"/>
 </segment>
 </net>
@@
 </segment>
 <segment>
-<pinref part="U$1" gate="G$1" pin="GPIO4(ADC2_0)"/>
-<wire x1="655.32" y1="-525.78" x2="665.48" y2="-525.78" width="0.1524" layer="91"/>
-<label x="665.48" y="-525.78" size="1.27" layer="95" xref="yes"/>
+<pinref part="U$1" gate="G$1" pin="GPIO14(ADC2_6/MTMSHSPI_SCK)"/>
+<wire x1="589.28" y1="-523.24" x2="584.2" y2="-523.24" width="0.1524" layer="91"/>
+<label x="584.2" y="-523.24" size="1.016" layer="95" rot="R180" xref="yes"/>
 </segment>
 </net>
@@
 </segment>
 <segment>
-<pinref part="U$1" gate="G$1" pin="GPIO17"/>
-<wire x1="655.32" y1="-520.7" x2="665.48" y2="-520.7" width="0.1524" layer="91"/>
-<label x="665.48" y="-520.7" size="1.27" layer="95" xref="yes"/>
+<pinref part="U$1" gate="G$1" pin="GPIO26(ADC2_9)"/>
+<wire x1="589.28" y1="-518.16" x2="584.2" y2="-518.16" width="0.1524" layer="91"/>
+<label x="584.2" y="-518.16" size="1.016" layer="95" rot="R180" xref="yes"/>
 </segment>
 </net>
@@
 </segment>
 <segment>
-<pinref part="U$1" gate="G$1" pin="GPIO0(ADC2_1)"/>
-<wire x1="655.32" y1="-528.32" x2="665.48" y2="-528.32" width="0.1524" layer="91"/>
-<label x="665.48" y="-528.32" size="1.27" layer="95" xref="yes"/>
+<pinref part="U$1" gate="G$1" pin="GPIO12(ADC2_5/MTDI/HSPI_MISO)"/>
+<wire x1="589.28" y1="-525.78" x2="584.2" y2="-525.78" width="0.1524" layer="91"/>
+<label x="584.2" y="-525.78" size="1.016" layer="95" rot="R180" xref="yes"/>
 </segment>
 </net>
@@
 </segment>
 <segment>
-<pinref part="U$1" gate="G$1" pin="GPIO16"/>
-<wire x1="655.32" y1="-523.24" x2="665.48" y2="-523.24" width="0.1524" layer="91"/>
-<label x="665.48" y="-523.24" size="1.27" layer="95" xref="yes"/>
+<pinref part="U$1" gate="G$1" pin="GPIO13(ADC2_4/MTCK/HSPI_MOSI)"/>
+<wire x1="589.28" y1="-530.86" x2="584.2" y2="-530.86" width="0.1524" layer="91"/>
+<label x="584.2" y="-530.86" size="1.016" layer="95" rot="R180" xref="yes"/>
 </segment>
 </net>
@@
 </segment>
 <segment>
-<pinref part="SERVO" gate="A" pin="2"/>
-<wire x1="640.08" y1="-449.58" x2="635" y2="-449.58" width="0.1524" layer="91"/>
-<label x="635" y="-449.58" size="1.27" layer="95" rot="R180" xref="yes"/>
+<pinref part="SERVO" gate="A" pin="1"/>
+<wire x1="640.08" y1="-447.04" x2="635" y2="-447.04" width="0.1524" layer="91"/>
+<label x="635" y="-447.04" size="1.27" layer="95" rot="R180" xref="yes"/>
 </segment>
 </net>
@@
 </segment>
 </net>
-<net name="IO27" class="0">
-<segment>
-<pinref part="U$1" gate="G$1" pin="GPIO27(ADC2_7)"/>
-<wire x1="589.28" y1="-520.7" x2="584.2" y2="-520.7" width="0.1524" layer="91"/>
-<label x="584.2" y="-520.7" size="1.27" layer="95" rot="R180" xref="yes"/>
-</segment>
-</net>
 <net name="IO25" class="0">
 <segment>
@@
 <net name="IO26" class="0">
 <segment>
-<pinref part="U$1" gate="G$1" pin="GPIO26(ADC2_9)"/>
-<wire x1="589.28" y1="-518.16" x2="584.2" y2="-518.16" width="0.1524" layer="91"/>
-<label x="584.2" y="-518.16" size="1.27" layer="95" rot="R180" xref="yes"/>
-</segment>
-<segment>
-<pinref part="SHALL" gate="A" pin="2"/>
-<wire x1="609.6" y1="-449.58" x2="604.52" y2="-449.58" width="0.1524" layer="91"/>
-<label x="604.52" y="-449.58" size="1.27" layer="95" rot="R180" xref="yes"/>
+<pinref part="SHALL" gate="A" pin="1"/>
+<wire x1="609.6" y1="-447.04" x2="604.52" y2="-447.04" width="0.1524" layer="91"/>
+<label x="604.52" y="-447.04" size="1.27" layer="95" rot="R180" xref="yes"/>
+</segment>
+<segment>
+<pinref part="U$1" gate="G$1" pin="GPIO32(ADC1_4)"/>
+<wire x1="589.28" y1="-510.54" x2="584.2" y2="-510.54" width="0.1524" layer="91"/>
+<label x="584.2" y="-510.54" size="1.27" layer="95" rot="R180" xref="yes"/>
 </segment>
 </net>
@@
 </segment>
 <segment>
-<pinref part="U$1" gate="G$1" pin="GPIO01(TX)"/>
-<wire x1="655.32" y1="-502.92" x2="665.48" y2="-502.92" width="0.1524" layer="91"/>
-<label x="665.48" y="-502.92" size="1.27" layer="95" xref="yes"/>
+<pinref part="U$1" gate="G$1" pin="GPIO17"/>
+<wire x1="655.32" y1="-520.7" x2="665.48" y2="-520.7" width="0.1524" layer="91"/>
+<label x="665.48" y="-520.7" size="1.27" layer="95" xref="yes"/>
 </segment>
 </net>
@@
 </segment>
 <segment>
-<pinref part="U$1" gate="G$1" pin="GPIO03(RX)"/>
-<wire x1="655.32" y1="-505.46" x2="665.48" y2="-505.46" width="0.1524" layer="91"/>
-<label x="665.48" y="-505.46" size="1.27" layer="95" xref="yes"/>
-</segment>
-</net>
+<pinref part="U$1" gate="G$1" pin="GPIO16"/>
+<wire x1="655.32" y1="-523.24" x2="665.48" y2="-523.24" width="0.1524" layer="91"/>
+<label x="665.48" y="-523.24" size="1.27" layer="95" xref="yes"/>
+</segment>
+</net>
